File: hardware/LED-Panel/led-strip-main-connector.brd (EAGLE design)
At the start: 96.2 x 41.9 mm, 27 parts, among them J1 1

Commit message: updating eagle files
Parts:
- turned SPARK_CORE to 90 degrees
Connections:
- removed net N$1 (its old number): STRIP-POS1.1, STRIP-POS2.1, STRIP-POS3.1, STRIP-POS4.1, STRIP-POS5.1, STRIP-POS6.1, STRIP-POS7.1, STRIP-POS8.1
- removed net N$2: STRIP-NEG1.1, STRIP-NEG2.1, STRIP-NEG3.1, STRIP-NEG4.1, STRIP-NEG5.1, STRIP-NEG6.1, STRIP-NEG7.1, STRIP-NEG8.1
- net N$5: now also STRIP-NEG1.1, STRIP-NEG2.1, STRIP-NEG3.1, STRIP-NEG4.1, STRIP-NEG5.1, STRIP-NEG6.1, STRIP-NEG7.1, STRIP-NEG8.1
- net N$6: now also STRIP-POS1.1, STRIP-POS2.1, STRIP-POS3.1, STRIP-POS4.1, STRIP-POS5.1, STRIP-POS6.1, STRIP-POS7.1, STRIP-POS8.1
Routing:
- net N$1 (its old number): track 207.6 -> 0.00 mm, vias 1 -> 0
- net N$2: track 168.7 -> 0.00 mm
- net N$6: track 0.00 -> 128.5 mm, vias 0 -> 1
- net N$5: track 0.00 -> 102.0 mm
- net N$1: track 104.9 -> 94.1 mm
Other:
- board text added: "BlinkyHat.com"
